File: muffboard.kicad_pcb (KiCad board)
At the start: 2 copper layers, 0 parts

Commit message: initial component placing on pcb
Parts:
- added C1: 100n, Capacitor_THT:C_Rect_L7.2mm_W2.5mm_P5.00mm_FKS2_FKP2_MKS2_MKP2, F.Cu at (107.8, 32.2)
- added C10: 470p, Capacitor_THT:C_Rect_L7.2mm_W2.5mm_P5.00mm_FKS2_FKP2_MKS2_MKP2, F.Cu at (105.7, 36.3)
- added C11: 4n, Capacitor_THT:C_Rect_L7.2mm_W2.5mm_P5.00mm_FKS2_FKP2_MKS2_MKP2, F.Cu at (97.9, 43.9)
- added C12: 10n, Capacitor_THT:C_Rect_L7.2mm_W2.5mm_P5.00mm_FKS2_FKP2_MKS2_MKP2, F.Cu at (107.8, 28.2)
- added C13: 100n, Capacitor_THT:C_Rect_L7.2mm_W2.5mm_P5.00mm_FKS2_FKP2_MKS2_MKP2, F.Cu at (73.2, 67.0)
- added C14: 100n, Capacitor_THT:C_Rect_L7.2mm_W2.5mm_P5.00mm_FKS2_FKP2_MKS2_MKP2, F.Cu at (97.0, 39.9)
- added C15: 100n, Capacitor_THT:C_Rect_L7.2mm_W2.5mm_P5.00mm_FKS2_FKP2_MKS2_MKP2, F.Cu at (97.0, 35.8)
- added C16: 100n, Capacitor_THT:C_Rect_L7.2mm_W2.5mm_P5.00mm_FKS2_FKP2_MKS2_MKP2, F.Cu at (51.7, 82.8)
- added C2: 100u, Capacitor_THT:CP_Radial_D6.3mm_P2.50mm, F.Cu at (76.8, 78.7)
- added C3: 470p, Capacitor_THT:C_Rect_L7.2mm_W2.5mm_P5.00mm_FKS2_FKP2_MKS2_MKP2, F.Cu at (91.8, 48.5)
- added C4: 100n, Capacitor_THT:C_Rect_L7.2mm_W2.5mm_P5.00mm_FKS2_FKP2_MKS2_MKP2, F.Cu at (67.1, 71.2)
- added C5: 100n, Capacitor_THT:C_Rect_L7.2mm_W2.5mm_P5.00mm_FKS2_FKP2_MKS2_MKP2, F.Cu at (67.1, 75.2)
- added C6: 47n, Capacitor_THT:C_Rect_L7.2mm_W2.5mm_P5.00mm_FKS2_FKP2_MKS2_MKP2, F.Cu at (91.8, 52.5)
- added C7: 470p, Capacitor_THT:C_Rect_L7.2mm_W2.5mm_P5.00mm_FKS2_FKP2_MKS2_MKP2, F.Cu at (116.5, 28.2)
- added C8: 100n, Capacitor_THT:C_Rect_L7.2mm_W2.5mm_P5.00mm_FKS2_FKP2_MKS2_MKP2, F.Cu at (60.4, 82.8)
- added C9: 47n, Capacitor_THT:C_Rect_L7.2mm_W2.5mm_P5.00mm_FKS2_FKP2_MKS2_MKP2, F.Cu at (83.5, 60.6)
- added D1: 1N4007, Diode_THT:D_DO-41_SOD81_P10.16mm_Horizontal, F.Cu at (51.7, 46.8)
- added D2: 1N4148, Diode_THT:D_DO-35_SOD27_P7.62mm_Horizontal, F.Cu at (38.4, 83.3)
- added D3: 1N4148, Diode_THT:D_DO-35_SOD27_P7.62mm_Horizontal, F.Cu at (96.7, 32.0)
- added D4: RED, LED_THT:LED_D3.0mm, F.Cu at (108.5, 44.3)
- added D5: RED, LED_THT:LED_D3.0mm, F.Cu at (100.3, 54.5)
- added D6: 1N4148, Diode_THT:D_DO-35_SOD27_P7.62mm_Horizontal, F.Cu at (51.4, 70.9)
- added D7: 1N4148, Diode_THT:D_DO-35_SOD27_P7.62mm_Horizontal, F.Cu at (27.6, 83.3)
- added D8: RED, LED_THT:LED_D3.0mm, F.Cu at (114.3, 38.8)
- added D9: RED, LED_THT:LED_D3.0mm, F.Cu at (92.0, 63.1)
- added J1: Conn_01x02, Connector_PinHeader_2.54mm:PinHeader_1x02_P2.54mm_Vertical, F.Cu at (125.7, 28.5)
- added J2: Conn_01x03, Connector_PinHeader_2.54mm:PinHeader_1x03_P2.54mm_Vertical, F.Cu at (87.6, 48.8)
- added J3: Conn_01x03, Connector_PinHeader_2.54mm:PinHeader_1x03_P2.54mm_Vertical, F.Cu at (62.9, 71.5)
- added Q1: BC547, Package_TO_SOT_THT:TO-92_Inline_Wide, F.Cu at (83.1, 65.9)
- added Q2: BC547, Package_TO_SOT_THT:TO-92_Inline_Wide, F.Cu at (75.5, 72.2)
- added Q3: BC547, Package_TO_SOT_THT:TO-92_Inline_Wide, F.Cu at (116.2, 33.5)
- added Q4: BC547, Package_TO_SOT_THT:TO-92_Inline_Wide, F.Cu at (100.2, 49.2)
- added Q5: BC547, Package_TO_SOT_THT:TO-92_Inline_Wide, F.Cu at (91.9, 57.8)
- added R1: 1M, Resistor_THT:R_Axial_DIN0207_L6.3mm_D2.5mm_P7.62mm_Horizontal, F.Cu at (65.3, 46.6)
- added R10: 470k, Resistor_THT:R_Axial_DIN0207_L6.3mm_D2.5mm_P7.62mm_Horizontal, F.Cu at (51.4, 78.8)
- added R11: 12k, Resistor_THT:R_Axial_DIN0207_L6.3mm_D2.5mm_P7.62mm_Horizontal, F.Cu at (86.8, 44.4)
- added R12: 150, Resistor_THT:R_Axial_DIN0207_L6.3mm_D2.5mm_P7.62mm_Horizontal, F.Cu at (62.2, 67.1)
- added R13: 8.2k, Resistor_THT:R_Axial_DIN0207_L6.3mm_D2.5mm_P7.62mm_Horizontal, F.Cu at (51.4, 50.9)
- added R14: 100k, Resistor_THT:R_Axial_DIN0207_L6.3mm_D2.5mm_P7.62mm_Horizontal, F.Cu at (75.1, 28.2)
- added R15: 470k, Resistor_THT:R_Axial_DIN0207_L6.3mm_D2.5mm_P7.62mm_Horizontal, F.Cu at (51.4, 59.0)
- added R16: 12k, Resistor_THT:R_Axial_DIN0207_L6.3mm_D2.5mm_P7.62mm_Horizontal, F.Cu at (51.4, 63.0)
- added R17: 150, Resistor_THT:R_Axial_DIN0207_L6.3mm_D2.5mm_P7.62mm_Horizontal, F.Cu at (75.1, 36.3)
- added R18: 33k, Resistor_THT:R_Axial_DIN0207_L6.3mm_D2.5mm_P7.62mm_Horizontal, F.Cu at (62.2, 50.9)
- added R19: 33k, Resistor_THT:R_Axial_DIN0207_L6.3mm_D2.5mm_P7.62mm_Horizontal, F.Cu at (85.9, 28.2)
- added R2: 33k, Resistor_THT:R_Axial_DIN0207_L6.3mm_D2.5mm_P7.62mm_Horizontal, F.Cu at (62.2, 63.0)
- added R20: 470k, Resistor_THT:R_Axial_DIN0207_L6.3mm_D2.5mm_P7.62mm_Horizontal, F.Cu at (85.9, 40.4)
- added R21: 47k, Resistor_THT:R_Axial_DIN0207_L6.3mm_D2.5mm_P7.62mm_Horizontal, F.Cu at (51.4, 55.0)
- added R22: 10k, Resistor_THT:R_Axial_DIN0207_L6.3mm_D2.5mm_P7.62mm_Horizontal, F.Cu at (76.1, 48.5)
- added R23: 390, Resistor_THT:R_Axial_DIN0207_L6.3mm_D2.5mm_P7.62mm_Horizontal, F.Cu at (75.1, 32.2)
- added R24: 470k, Resistor_THT:R_Axial_DIN0207_L6.3mm_D2.5mm_P7.62mm_Horizontal, F.Cu at (62.2, 55.0)
- added R25: 100k, Resistor_THT:R_Axial_DIN0207_L6.3mm_D2.5mm_P7.62mm_Horizontal, F.Cu at (75.1, 40.4)
- added R26: 12k, Resistor_THT:R_Axial_DIN0207_L6.3mm_D2.5mm_P7.62mm_Horizontal, F.Cu at (85.9, 32.2)
- added R27: 2.7k, Resistor_THT:R_Axial_DIN0207_L6.3mm_D2.5mm_P7.62mm_Horizontal, F.Cu at (62.2, 59.0)
- added R3: 100k, Resistor_THT:R_Axial_DIN0207_L6.3mm_D2.5mm_P7.62mm_Horizontal, F.Cu at (85.9, 36.3)
- added R4: 470k, Resistor_THT:R_Axial_DIN0207_L6.3mm_D2.5mm_P7.62mm_Horizontal, F.Cu at (96.7, 28.2)
- added R5: 15k, Resistor_THT:R_Axial_DIN0207_L6.3mm_D2.5mm_P7.62mm_Horizontal, F.Cu at (72.9, 52.5)
- added R6: 150, Resistor_THT:R_Axial_DIN0207_L6.3mm_D2.5mm_P7.62mm_Horizontal, F.Cu at (76.1, 44.4)
- added R7: 1k, Resistor_THT:R_Axial_DIN0207_L6.3mm_D2.5mm_P7.62mm_Horizontal, F.Cu at (51.4, 67.1)
- added R8: 8.2k, Resistor_THT:R_Axial_DIN0207_L6.3mm_D2.5mm_P7.62mm_Horizontal, F.Cu at (51.4, 74.7)
- added R9: 100k, Resistor_THT:R_Axial_DIN0207_L6.3mm_D2.5mm_P7.62mm_Horizontal, F.Cu at (72.9, 56.5)
- added RV1: 100k, Potentiometer_THT:Potentiometer_Omeg_PC16BU_Vertical, B.Cu at (141.0, 86.1)
- added RV2: 100k, Potentiometer_THT:Potentiometer_Omeg_PC16BU_Vertical, B.Cu at (141.0, 61.1)
- added RV3: 100k, Potentiometer_THT:Potentiometer_Omeg_PC16BU_Vertical, B.Cu at (172.0, 86.6)
- added RV4: 100k, Potentiometer_THT:Potentiometer_Omeg_PC16BU_Vertical, B.Cu at (172.0, 61.1)
- added SW1: SW_DPDT_x2, Button_Switch_THT:SW_E-Switch_EG1271_DPDT, B.Cu at (149.9, 76.6)
