File: muffboard.kicad_pcb (KiCad board)
At the start: 2 copper layers, 65 parts, among them J1 Conn_01x02, J2 Conn_01x03, J3 Conn_01x03, Q1 BC547, Q2 BC547, Q3 BC547, Q4 BC547, Q5 BC547, SW1 SW_DPDT_x2

Commit message: finished board (de estoura)
Parts:
- moved D1 134.9 mm to (161.0, 125.8)
- moved D7 132.9 mm to (159.9, 96.4), turned to 180 degrees
- moved R7 132.5 mm to (171.7, 122.6), turned to 90 degrees
- moved R21 120.9 mm to (167.3, 89.4), turned to -90 degrees
- moved R6 117.5 mm to (171.7, 112.6), turned to 90 degrees
- moved J3 116.4 mm to (163.8, 129.6), turned to 90 degrees
- moved R23 114.1 mm to (173.9, 89.4), turned to -90 degrees
- moved R3 113.3 mm to (168.3, 114.0), turned to 90 degrees
- moved R5 110.8 mm to (172.1, 102.0), turned to 180 degrees
- moved C16 110.1 mm to (161.7, 85.8), turned to 90 degrees
- moved D2 106.6 mm to (144.5, 93.6), turned to 180 degrees
- moved J1 105.0 mm to (154.1, 129.6), turned to -90 degrees
- moved R4 103.9 mm to (165.1, 106.4), turned to -90 degrees
- moved D6 103.4 mm to (152.2, 93.6)
- moved R10 102.1 mm to (147.2, 113.9), turned to 90 degrees
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Connections:
- net Net-(C14-Pad1) renamed /volume_pot1
- net Net-(C16-Pad2) renamed /boost_pot1
- net VBUS renamed VCC
- C11 pad 2: /1,27 -> /q3c
- C15 pad 2: Net-(C15-Pad2) -> /q5b
- C16 pad 1: Net-(C16-Pad1) -> /q5c
- Q4 pad 1: Net-(C16-Pad1) -> /q4c
- Q4 pad 2: Net-(C15-Pad2) -> /q4b
- Q4 pad 3: Net-(Q4-Pad3) -> /q4e
- Q5 pad 1: /q4c -> /q5c
- Q5 pad 2: /q4b -> /q5b
- Q5 pad 3: /q4e -> /q5e
- R18 pad 2: /1,27 -> /q3c
- R20 pad 2: Net-(C15-Pad2) -> /q5b
- R21 pad 1: Net-(C15-Pad2) -> /q5b
- R22 pad 2: Net-(C16-Pad1) -> /q5c
- R23 pad 1: Net-(Q4-Pad3) -> /q5e
Routing:
- net VCC: track 0.00 -> 155.7 mm
- net /boost_out: track 0.00 -> 65.4 mm
- net /q3c: track 0.00 -> 63.6 mm
- net /q2c: track 0.00 -> 43.8 mm, vias 0 -> 1
- net /q1b: track 0.00 -> 36.8 mm
- net /boost_in: track 0.00 -> 35.2 mm
- net /q2b: track 0.00 -> 31.2 mm
- net /q1c: track 0.00 -> 24.3 mm
- net /q4b: track 0.00 -> 21.8 mm
- net Net-(C5-Pad2): track 0.00 -> 21.7 mm
- net /q3b: track 0.00 -> 20.8 mm
- net /clipmod1in: track 0.00 -> 18.6 mm
- net /q4c: track 0.00 -> 17.6 mm
- net /Input: track 0.00 -> 16.1 mm
- net /clipmod2in: track 0.00 -> 16.0 mm
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- added copper zone on B.Cu, net GND
Other:
- board outline added: 57 x 59.2 mm

Commit message: rev 1.0 board
Other:
- board size 57 x 59.2 mm -> 60 x 59.2 mm
- board text added: "+9V"
- board text added: "Boost 1 2 3"
- board text added: "GND"
- board text added: "Input"
- board text added: "Output"
- board text added: "Sustain 3 2 1"
- board text added: "Tone 1 2 3"
- board text added: "Volume 3 2 1"
- board text added: "boost_in"
- board text added: "boost_out"
- board text added: "jpais"
- board text added: "muffler delete rev 1.0"
Changed lines of the file:
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@@
     (property "Sheetname" "")
     (attr through_hole)
-    (fp_text reference "SW1" (at 2.5 1.65 90) (layer "B.SilkS")
+    (fp_text reference "SW1" (at -3.16 -1.49 180) (layer "B.SilkS")
       (effects (font (size 1 1) (thickness 0.15)) (justify mirror))
     )
@@
     (property "Sheetname" "")
     (attr through_hole)
-    (fp_text reference "RV3" (at 0.1 14.6 90) (layer "B.SilkS")
+    (fp_text reference "RV3" (at 0.1 14.6 90) (layer "B.SilkS") hide
       (effects (font (size 1 1) (thickness 0.15)) (justify mirror))
     )
@@
       (effects (font (size 1 1) (thickness 0.15)) (justify mirror))
     )
-    (fp_text user "${REFERENCE}" (at 2.75 5) (layer "B.Fab")
-      (effects (font (size 1 1) (thickness 0.15)) (justify mirror))
-    )
-    (fp_line (start 1.63 -3.57) (end 12.55 -3.57) (layer "B.SilkS") (width 0.12))
-    (fp_line (start 1.63 13.57) (end 12.55 13.57) (layer "B.SilkS") (width 0.12))
-    (fp_line (start 1.63 13.57) (end 1.63 -3.57) (layer "B.SilkS") (width 0.12))
-    (fp_circle (center 12.55 5) (end 21.12 5) (layer "B.SilkS") (width 0.12) (fill none))
+    (fp_text user "${REFERENCE}" (at 2.75 5 180) (layer "B.Fab")
+      (effects (font (size 1 1) (thickness 0.15)) (justify mirror))
+    )
     (fp_line (start 21.25 13.7) (end -1.45 13.7) (layer "B.CrtYd") (width 0.05))
     (fp_line (start -1.45 -3.7) (end 21.25 -3.7) (layer "B.CrtYd") (width 0.05))
@@
     (property "Sheetname" "")
     (attr through_hole)
-    (fp_text reference "RV4" (at 0.2 -4.5 90) (layer "B.SilkS")
-      (effects (font (size 1 1) (thickness 0.15)) (justify mirror))
-    )
-    (fp_text value "100k" (at 9.915 -4.7 90) (layer "B.Fab")
+    (fp_text reference "RV4" (at 0.2 -4.5 270) (layer "B.SilkS") hide
+      (effects (font (size 1 1) (thickness 0.15)) (justify mirror))
+    )
+    (fp_text value "100k" (at 9.915 -4.7 270) (layer "B.Fab")
       (effects (font (size 1 1) (thickness 0.15)) (justify mirror))
     )
@@
       (effects (font (size 1 1) (thickness 0.15)) (justify mirror))
     )
-    (fp_line (start 1.63 13.57) (end 12.55 13.57) (layer "B.SilkS") (width 0.12))
-    (fp_line (start 1.63 13.57) (end 1.63 -3.57) (layer "B.SilkS") (width 0.12))
-    (fp_line (start 1.63 -3.57) (end 12.55 -3.57) (layer "B.SilkS") (width 0.12))
-    (fp_circle (center 12.55 5) (end 21.12 5) (layer "B.SilkS") (width 0.12) (fill none))
     (fp_line (start 21.25 -3.7) (end 21.25 13.7) (layer "B.CrtYd") (width 0.05))
     (fp_line (start 21.25 13.7) (end -1.45 13.7) (layer "B.CrtYd") (width 0.05))
@@
     (property "Sheetname" "")
     (attr through_hole)
-    (fp_text reference "RV1" (at 0 -4.4 90) (layer "B.SilkS")
-      (effects (font (size 1 1) (thickness 0.15)) (justify mirror))
-    )
-    (fp_text value "100k" (at 9.915 -4.7 90) (layer "B.Fab")
+    (fp_text reference "RV1" (at 0 -4.4 270) (layer "B.SilkS") hide
+      (effects (font (size 1 1) (thickness 0.15)) (justify mirror))
+    )
+    (fp_text value "100k" (at 9.915 -4.7 270) (layer "B.Fab")
       (effects (font (size 1 1) (thickness 0.15)) (justify mirror))
     )
@@
       (effects (font (size 1 1) (thickness 0.15)) (justify mirror))
     )
-    (fp_line (start 1.63 13.57) (end 1.63 -3.57) (layer "B.SilkS") (width 0.12))
-    (fp_line (start 1.63 -3.57) (end 12.55 -3.57) (layer "B.SilkS") (width 0.12))
-    (fp_line (start 1.63 13.57) (end 12.55 13.57) (layer "B.SilkS") (width 0.12))
-    (fp_circle (center 12.55 5) (end 21.12 5) (layer "B.SilkS") (width 0.12) (fill none))
     (fp_line (start -1.45 13.7) (end -1.45 -3.7) (layer "B.CrtYd") (width 0.05))
     (fp_line (start 21.25 13.7) (end -1.45 13.7) (layer "B.CrtYd") (width 0.05))
@@
     (property "Sheetname" "")
     (attr through_hole)
-    (fp_text reference "RV2" (at -0.1 14.5 90) (layer "B.SilkS")
+    (fp_text reference "RV2" (at -0.1 14.5 90) (layer "B.SilkS") hide
       (effects (font (size 1 1) (thickness 0.15)) (justify mirror))
     )
@@
       (effects (font (size 1 1) (thickness 0.15)) (justify mirror))
     )
-    (fp_text user "${REFERENCE}" (at 2.75 5) (layer "B.Fab")
-      (effects (font (size 1 1) (thickness 0.15)) (justify mirror))
-    )
-    (fp_line (start 1.63 13.57) (end 1.63 -3.57) (layer "B.SilkS") (width 0.12))
-    (fp_line (start 1.63 -3.57) (end 12.55 -3.57) (layer "B.SilkS") (width 0.12))
-    (fp_line (start 1.63 13.57) (end 12.55 13.57) (layer "B.SilkS") (width 0.12))
-    (fp_circle (center 12.55 5) (end 21.12 5) (layer "B.SilkS") (width 0.12) (fill none))
+    (fp_text user "${REFERENCE}" (at 2.75 5 180) (layer "B.Fab")
+      (effects (font (size 1 1) (thickness 0.15)) (justify mirror))
+    )
     (fp_line (start 21.25 13.7) (end -1.45 13.7) (layer "B.CrtYd") (width 0.05))
     (fp_line (start 21.25 -3.7) (end 21.25 13.7) (layer "B.CrtYd") (width 0.05))
@@
   )
   (gr_arc (start 175.9 72.8) (mid 177.031371 73.268629) (end 177.5 74.4) (layer "Edge.Cuts") (width 0.05))
-  (gr_arc (start 122.1 132) (mid 120.968629 131.531371) (end 120.5 130.4) (layer "Edge.Cuts") (width 0.05))
-  (gr_line (start 122.1 132) (end 175.9 132) (layer "Edge.Cuts") (width 0.05))
-  (gr_arc (start 120.5 74.4) (mid 120.968629 73.268629) (end 122.1 72.8) (layer "Edge.Cuts") (width 0.05))
-  (gr_line (start 120.5 74.4) (end 120.5 130.4) (layer "Edge.Cuts") (width 0.05))
+  (gr_arc (start 119.131371 132) (mid 118 131.531371) (end 117.531371 130.4) (layer "Edge.Cuts") (width 0.05))
+  (gr_line (start 119.131371 132) (end 175.9 132) (layer "Edge.Cuts") (width 0.05))
+  (gr_arc (start 117.531371 74.4) (mid 118 73.268629) (end 119.131371 72.8) (layer "Edge.Cuts") (width 0.05))
+  (gr_line (start 117.531371 74.4) (end 117.531371 130.4) (layer "Edge.Cuts") (width 0.05))
   (gr_arc (start 177.5 130.4) (mid 177.031371 131.531371) (end 175.9 132) (layer "Edge.Cuts") (width 0.05))
   (gr_line (start 177.5 74.4) (end 177.5 129) (layer "Edge.Cuts") (width 0.05))
   (gr_line (start 177.5 130.4) (end 177.5 129) (layer "Edge.Cuts") (width 0.05))
-  (gr_line (start 122.1 72.8) (end 175.9 72.8) (layer "Edge.Cuts") (width 0.05))
+  (gr_line (start 119.131371 72.8) (end 175.9 72.8) (layer "Edge.Cuts") (width 0.05))
+  (gr_text "GND\n" (at 166.3 131.4) (layer "B.SilkS")
+    (effects (font (size 0.7 0.7) (thickness 0.15)) (justify mirror))
+  )
+  (gr_text "boost_out" (at 170.6 131.4) (layer "B.SilkS")
+    (effects (font (size 0.7 0.7) (thickness 0.15)) (justify mirror))
+  )
+  (gr_text "GND\n" (at 151.5 131.3) (layer "B.SilkS")
+    (effects (font (size 0.7 0.7) (thickness 0.15)) (justify mirror))
+  )
+  (gr_text "Sustain 3 2 1\n" (at 163.5 120) (layer "B.SilkS")
+    (effects (font (size 1 1) (thickness 0.15)) (justify mirror))
+  )
+  (gr_text "Output\n" (at 131.5 131.3) (layer "B.SilkS")
+    (effects (font (size 0.7 0.7) (thickness 0.15)) (justify mirror))
+  )
+  (gr_text "Boost 1 2 3\n" (at 163.5 74) (layer "B.SilkS")
+    (effects (font (size 1 1) (thickness 0.15)) (justify mirror))
+  )
+  (gr_text "Input" (at 137.9 131.3) (layer "B.SilkS")
+    (effects (font (size 0.7 0.7) (thickness 0.15)) (justify mirror))
+  )
+  (gr_text "Volume 3 2 1" (at 131.8 120) (layer "B.SilkS")
+    (effects (font (size 1 1) (thickness 0.15)) (justify mirror))
+  )
+  (gr_text "boost_in" (at 162.2 131.4) (layer "B.SilkS")
+    (effects (font (size 0.7 0.7) (thickness 0.15)) (justify mirror))
+  )
+  (gr_text "Tone 1 2 3" (at 131.5 74) (layer "B.SilkS")
+    (effects (font (size 1 1) (thickness 0.15)) (justify mirror))
+  )
+  (gr_text "+9V" (at 154.3 131.3) (layer "B.SilkS")
+    (effects (font (size 0.7 0.7) (thickness 0.15)) (justify mirror))
+  )
+  (gr_text "GND\n" (at 134.9 131.3) (layer "B.SilkS")
+    (effects (font (size 0.7 0.7) (thickness 0.15)) (justify mirror))
+  )
+  (gr_text "muffler delete rev 1.0" (at 119.75 112.25 90) (layer "F.SilkS")
+    (effects (font (size 1.5 1.5) (thickness 0.15)))
+  )
+  (gr_text "jpais" (at 119.75 127.75 90) (layer "F.SilkS")
+    (effects (font (size 1 1) (thickness 0.15)))
+  )
   (segment (start 149.919511 123.919511) (end 164.129403 123.919511) (width 0.3) (layer "F.Cu") (net 1))
   (segment (start 165.1 122.948914) (end 165.1 117.96) (width 0.3) (layer "F.Cu") (net 1))
@@
   (segment (start 161.7 80.8) (end 166 76.5) (width 0.3) (layer "F.Cu") (net 38))
   (segment (start 166 76.5) (end 168.5 76.5) (width 0.3) (layer "F.Cu") (net 38))
-  (segment (start 161.7 80.8) (end 161.9 80.6) (width 0.3) (layer "B.Cu") (net 38))
   (zone (net 4) (net_name "GND") (layer "B.Cu") (hatch edge 0.508)
     (connect_pads (clearance 0.508))
@@
         (xy 177.5 72.8)
         (xy 177.5 132)
-        (xy 120.5 132)
-        (xy 120.5 72.8)
+        (xy 117.5 132)
+        (xy 117.5 72.8)
       )
     )
