File: muffboard.kicad_sch (KiCad schematic)
At the start: 65 parts, among them J1 Conn_01x02, J2 Conn_01x03, J3 Conn_01x03, Q1 BC547, Q2 BC547, Q3 BC547, Q4 BC547, Q5 BC547, SW1 SW_DPDT_x2

Commit message: initial component placing on pcb
Parts:
- SW1: footprint (none) -> Button_Switch_THT:SW_E-Switch_EG1271_DPDT
Other:
- note added: "Selectable clipping modes using a switch, allowing the player to choose between a classic big muff sound, or a more "overdrivy" sound using LED clipping"
- note removed: "Selectable clipping modes using a switch, allowing the player to choose between a classic big muff sound, or a more overdrive sound using LED clipping"
- moved on the sheet: D2, D3, D4, D5, D6, D7, D8, D9, SW1A, SW1B

Commit message: finished board (de estoura)
Parts:
- renumbered Q5 to Q4, Q4 to Q5
Connections:
- net 1,27 is gone; now on net q3c: C11.2, R18.2
- net volume_pot1: now reaches C14.1, RV4.1
- net q5c: now reaches C16.1, Q5.1 (C), R22.2
- net q5b: now reaches C15.2, Q5.2 (B), R20.2, R21.1
- net q5e: now reaches Q5.3 (E), R23.1
- net boost_pot1: now reaches C16.2, RV3.1
- net VBUS renamed VCC
Changed lines of the file:
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@@
-    (stroke (width 0) (type default) (color 0 0 0 0))
-  )
-  (wire (pts (xy 68.58 163.83) (xy 68.58 166.37))
     (stroke (width 0) (type default) (color 0 0 0 0))
   )
@@
     (effects (font (size 1.27 1.27)) (justify left bottom))
   )
+  (label "q5c" (at 302.26 172.72 0)
+    (effects (font (size 1 1)) (justify left bottom))
+  )
   (label "q4c" (at 331.47 83.82 0)
     (effects (font (size 1.27 1.27)) (justify left bottom))
@@
     (effects (font (size 1 1)) (justify right bottom))
   )
-  (label "1,27" (at 254 81.28 0)
+  (label "q3c" (at 254 81.28 0)
     (effects (font (size 1 1)) (justify left bottom))
   )
@@
     (effects (font (size 1 1)) (justify left bottom))
   )
+  (label "boost_pot1" (at 320.04 175.26 0)
+    (effects (font (size 0.8 0.8)) (justify left bottom))
+  )
   (label "q1e" (at 99.06 101.6 0)
     (effects (font (size 1.27 1.27)) (justify left bottom))
@@
     (effects (font (size 1.27 1.27)) (justify left bottom))
   )
+  (label "q5e" (at 302.26 186.69 0)
+    (effects (font (size 1 1)) (justify left bottom))
+  )
   (label "boost_in" (at 127 175.26 180)
     (effects (font (size 1.27 1.27)) (justify right bottom))
@@
     (effects (font (size 0.8 0.8)) (justify left bottom))
   )
+  (label "volume_pot1" (at 350.52 83.82 0)
+    (effects (font (size 0.8 0.8)) (justify left bottom))
+  )
   (label "q2c" (at 198.12 165.1 0)
     (effects (font (size 1.27 1.27)) (justify left bottom))
@@
   (label "q3c" (at 245.11 92.71 180)
     (effects (font (size 1.27 1.27)) (justify right bottom))
+  )
+  (label "q5b" (at 292.1 179.07 0)
+    (effects (font (size 1 1)) (justify left bottom))
   )
   (label "boost_out" (at 127 180.34 180)
@@
   (symbol (lib_id "Transistor_BJT:BC547") (at 327.66 91.44 0) (unit 1)
     (in_bom yes) (on_board yes)
-    (property "Reference" "Q5" (id 0) (at 332.5114 90.2716 0)
+    (property "Reference" "Q4" (id 0) (at 332.5114 90.2716 0)
       (effects (font (size 1.27 1.27)) (justify left))
     )
@@
   (symbol (lib_id "Transistor_BJT:BC547") (at 299.72 179.07 0) (unit 1)
     (in_bom yes) (on_board yes) (fields_autoplaced)
-    (property "Reference" "Q4" (id 0) (at 304.5714 178.1615 0)
-      (effects (font (size 1.27 1.27)) (justify left))
-    )
-    (property "Value" "BC547" (id 1) (at 304.5714 180.9366 0)
+    (property "Reference" "Q5" (id 0) (at 304.5714 178.2353 0)
+      (effects (font (size 1.27 1.27)) (justify left))
+    )
+    (property "Value" "BC547" (id 1) (at 304.5714 180.7722 0)
       (effects (font (size 1.27 1.27)) (justify left))
     )
@@
     (pin "1")
   )
-  (symbol (lib_id "power:VBUS") (at 68.58 163.83 0) (unit 1)
-    (in_bom yes) (on_board yes) (fields_autoplaced)
-    (property "Reference" "#PWR02" (id 0) (at 68.58 167.64 0)
-      (effects (font (size 1.27 1.27)) hide)
-    )
-    (property "Value" "VBUS" (id 1) (at 68.58 160.2255 0))
-    (property "Footprint" "" (id 2) (at 68.58 163.83 0)
-      (effects (font (size 1.27 1.27)) hide)
-    )
-    (property "Datasheet" "" (id 3) (at 68.58 163.83 0)
-      (effects (font (size 1.27 1.27)) hide)
-    )
-    (pin "1")
-  )
   (symbol (lib_id "power:GND") (at 218.44 118.11 0) (unit 1)
     (in_bom yes) (on_board yes)
@@
       (reference "#PWR01") (unit 1) (value "GND") (footprint "")
     )
-    (path "/74f20975-b791-4740-8a7d-cea55a2ffbbe"
-      (reference "#PWR02") (unit 1) (value "VBUS") (footprint "")
-    )
     (path "/00000000-0000-0000-0000-000061be6107"
       (reference "#PWR03") (unit 1) (value "GND") (footprint "")
@@
       (reference "Q3") (unit 1) (value "BC547") (footprint "Package_TO_SOT_THT:TO-92_Inline_Wide")
     )
+    (path "/00000000-0000-0000-0000-000061467e09"
+      (reference "Q4") (unit 1) (value "BC547") (footprint "Package_TO_SOT_THT:TO-92_Inline_Wide")
+    )
     (path "/410def68-8b62-4888-9363-5c9e7c3dbfbc"
-      (reference "Q4") (unit 1) (value "BC547") (footprint "Package_TO_SOT_THT:TO-92_Inline_Wide")
-    )
-    (path "/00000000-0000-0000-0000-000061467e09"
       (reference "Q5") (unit 1) (value "BC547") (footprint "Package_TO_SOT_THT:TO-92_Inline_Wide")
     )
